File: PDSU.kicad_sch (KiCad schematic)
At the start: 34 parts, among them J1 USB_C_Receptacle, J2 Conn_01x04, SW1 ON/OFF, U1 NCP1117-3.3_SOT223, U2 W25Q128JVS, U3 RP2040, Y1 ABM8-272-T3

Commit message: this is probably a fire hazard
Parts:
- removed C1, C4: 10u, Capacitor_SMD:C_0805_2012Metric, symbol Device:C
- removed J1: USB_C_Receptacle, Components:USB-C_SMD-TYPE-C-31-M-12, symbol Connector:USB_C_Receptacle
- removed R8, R9: 5.1k, Resistor_SMD:R_0402_1005Metric, symbol Device:R
- removed SW1: ON/OFF, Components:SW-SMD_XDMK-12C01-25, symbol XMDK-12C01-25:XDMK-12C01-25
- removed U1: NCP1117-3.3_SOT223, Package_TO_SOT_SMD:SOT-223-3_TabPin2, symbol Regulator_Linear:NCP1117-3.3_SOT223
Connections:
- no-connect marks 2 -> 0
Other:
- note removed: "Power"
- moved on the sheet: C10, C11, C12, C13, C14, C15, C16, C17, C6, C7, C8, C9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

Commit message: fire hazard!!!
Parts:
- removed J2: Conn_01x04, Components:SSD1306-0.91-OLED-4pin-128x32, symbol Connector_Generic:Conn_01x04
Connections:
- no-connect marks 0 -> 6
Other:
- added sheet PowerInput1 (PowerInput.kicad_sch)
- added sheet PowerInput2 (PowerInput.kicad_sch)
- added sheet PowerInput3 (PowerInput.kicad_sch)
- sheet PowerInput ports: added ALERT, GND, MCU_RESET, USB_D+, USB_D-, VOUT, V_MCU; removed none
- note removed: "OLED"
- moved on the sheet: C10, C11, C12, C13, C14, C15, C16, C17, C2, C3, C5, C6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
